File: Ideal Diode.kicad_sch (KiCad schematic)
At the start: 5 parts, among them Q3 MBT3906DW1, Q4 AO3401A

Commit message: Lots more routing and placement
Parts:
- C34: renamed from C35; footprint Capacitor_SMD:C_0402_1005Metric -> (none)
- R7: renamed from R9; footprint Resistor_SMD:R_0402_1005Metric -> (none)
- R8: renamed from R10; footprint Resistor_SMD:R_0402_1005Metric -> (none)
- renumbered Q3 to Q1, Q4 to Q2
Changed lines of the file:
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@@
 		(dnp no)
 		(fields_autoplaced yes)
-		(property "Reference" "R9"
+		(property "Reference" "R7"
 			(at 123.19 92.7099 0)
 			(show_name no)
@@
 			)
 		)
-		(property "Footprint" "Resistor_SMD:R_0402_1005Metric"
+		(property "Footprint" ""
 			(at 120.65 93.98 0)
 			(hide yes)
@@
 				(path "/00fce685-3911-4226-b2b0-c3fe2c89695c/7e7146d4-8a9f-4d35-96ce-85591b6e7d18"
 					(reference "R7")
-					(unit 1)
-				)
-			)
-			(project "Ideal Diode"
-				(path "/60a677a9-44fb-43ad-b21f-999b25bc2992"
-					(reference "R9")
 					(unit 1)
 				)
@@
 		(in_pos_files yes)
 		(dnp no)
-		(property "Reference" "Q3"
+		(property "Reference" "Q1"
 			(at 134.62 88.9001 0)
 			(show_name no)
@@
 				(path "/00fce685-3911-4226-b2b0-c3fe2c89695c/7e7146d4-8a9f-4d35-96ce-85591b6e7d18"
 					(reference "Q1")
-					(unit 2)
-				)
-			)
-			(project "Ideal Diode"
-				(path "/60a677a9-44fb-43ad-b21f-999b25bc2992"
-					(reference "Q3")
 					(unit 2)
 				)
@@
 		(dnp no)
 		(fields_autoplaced yes)
-		(property "Reference" "R10"
+		(property "Reference" "R8"
 			(at 160.02 92.7099 0)
 			(show_name no)
@@
 			)
 		)
-		(property "Footprint" "Resistor_SMD:R_0402_1005Metric"
+		(property "Footprint" ""
 			(at 157.48 93.98 0)
 			(hide yes)
@@
 				(path "/00fce685-3911-4226-b2b0-c3fe2c89695c/7e7146d4-8a9f-4d35-96ce-85591b6e7d18"
 					(reference "R8")
-					(unit 1)
-				)
-			)
-			(project "Ideal Diode"
-				(path "/60a677a9-44fb-43ad-b21f-999b25bc2992"
-					(reference "R10")
 					(unit 1)
 				)
@@
 		(dnp no)
 		(fields_autoplaced yes)
-		(property "Reference" "Q4"
+		(property "Reference" "Q2"
 			(at 148.59 60.96 90)
 			(show_name no)
@@
 				(path "/00fce685-3911-4226-b2b0-c3fe2c89695c/7e7146d4-8a9f-4d35-96ce-85591b6e7d18"
 					(reference "Q2")
-					(unit 1)
-				)
-			)
-			(project "Ideal Diode"
-				(path "/60a677a9-44fb-43ad-b21f-999b25bc2992"
-					(reference "Q4")
 					(unit 1)
 				)
@@
 		(in_pos_files yes)
 		(dnp no)
-		(property "Reference" "Q3"
+		(property "Reference" "Q1"
 			(at 106.68 86.3599 0)
 			(show_name no)
@@
 				(path "/00fce685-3911-4226-b2b0-c3fe2c89695c/7e7146d4-8a9f-4d35-96ce-85591b6e7d18"
 					(reference "Q1")
-					(unit 1)
-				)
-			)
-			(project "Ideal Diode"
-				(path "/60a677a9-44fb-43ad-b21f-999b25bc2992"
-					(reference "Q3")
 					(unit 1)
 				)
@@
 		(in_pos_files yes)
 		(dnp no)
-		(property "Reference" "C35"
+		(property "Reference" "C34"
 			(at 92.202 71.12 0)
 			(show_name no)
@@
 			)
 		)
-		(property "Footprint" "Capacitor_SMD:C_0402_1005Metric"
+		(property "Footprint" ""
 			(at 99.06 72.39 0)
 			(hide yes)
@@
 				(path "/00fce685-3911-4226-b2b0-c3fe2c89695c/7e7146d4-8a9f-4d35-96ce-85591b6e7d18"
 					(reference "C34")
-					(unit 1)
-				)
-			)
-			(project "Ideal Diode"
-				(path "/60a677a9-44fb-43ad-b21f-999b25bc2992"
-					(reference "C35")
 					(unit 1)
 				)
@@
 		(dnp no)
 		(fields_autoplaced yes)
-		(property "Reference" "#PWR064"
+		(property "Reference" "#PWR061"
 			(at 120.65 102.87 0)
 			(hide yes)
@@
 				(path "/00fce685-3911-4226-b2b0-c3fe2c89695c/7e7146d4-8a9f-4d35-96ce-85591b6e7d18"
 					(reference "#PWR061")
-					(unit 1)
-				)
-			)
-			(project "Ideal Diode"
-				(path "/60a677a9-44fb-43ad-b21f-999b25bc2992"
-					(reference "#PWR064")
 					(unit 1)
 				)
@@
 		(dnp no)
 		(fields_autoplaced yes)
-		(property "Reference" "#PWR065"
+		(property "Reference" "#PWR062"
 			(at 157.48 102.87 0)
 			(hide yes)
@@
 				(path "/00fce685-3911-4226-b2b0-c3fe2c89695c/7e7146d4-8a9f-4d35-96ce-85591b6e7d18"
 					(reference "#PWR062")
-					(unit 1)
-				)
-			)
-			(project "Ideal Diode"
-				(path "/60a677a9-44fb-43ad-b21f-999b25bc2992"
-					(reference "#PWR065")
 					(unit 1)
 				)
@@
 		(dnp no)
 		(fields_autoplaced yes)
-		(property "Reference" "#PWR063"
+		(property "Reference" "#PWR060"
 			(at 99.06 81.28 0)
 			(hide yes)
@@
 				)
 			)
-			(project "Ideal Diode"
-				(path "/60a677a9-44fb-43ad-b21f-999b25bc2992"
-					(reference "#PWR063")
-					(unit 1)
-				)
-			)
-		)
-	)
-	(sheet_instances
-		(path "/"
-			(page "1")
-		)
-	)
-	(embedded_fonts no)
+		)
+	)
 )
